Commit message: add SensorDataPublisher to simulation

File: base_station/roar/urdf/roar.urdf (robot description, URDF)
Before this commit: robot roar, 11 links, 10 joints
Joints:
- joint bogie_lhs_joint: type fixed -> continuous
- joint bogie_rhs_joint: type fixed -> continuous

Commit message: old filter design

File: base_station/roar/urdf/roar.urdf (robot description, URDF)
Before this commit: robot roar, 11 links, 10 joints
Joints:
- joint bogie_lhs_joint: type continuous -> fixed
- joint bogie_rhs_joint: type continuous -> fixed
